File: flight computer/horizon.kicad_pcb (KiCad board)
At the start: 4 copper layers, 50.8 x 100 mm, 174 parts, among them J1 Micro_SD_Card_Det1, J10 Conn_01x02_Pin, J11 USB_C_Receptacle_USB2.0_16P, J12 Conn_01x04, J13 1x3 servo, J14 1x3 servo, J15 arming terminal, J16 arming terminal, J17 H9161TR-ND, J18 Conn_02x03_Counter_Clockwise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

Commit message: magic
Parts:
- Y1: value Crystal -> 32 kHZ
